File: esp-led-box.sch (KiCad schematic (older format))
At the start: 68 parts, among them IC1 CP2105-F01-GMR, J1 Conn_01x03, J2 Conn_01x03_Female, J3 Conn_01x02_Female, J4 USB_B_Micro, Q1 BSS138, Q10 Q_PMOS_DGS, Q11 Q_PMOS_DGS, Q12 Q_NMOS_DGS, Q13 Q_PMOS_DGS, Q14 S8050, Q15 S8050, Q2 Q_NMOS, Q3 Q_DUAL_PMOS_G1S2G2D2S1D1, Q4 Q_P, Q5 Q_PMOS_DGS, Q6 Q_PMOS_DGS, Q7 Q_NMOS_DGS, Q8 Q_PMOS_DGS, Q9 Q_PMOS_DGS, U1 MP2307, U2 LM3940, U3 ESP-12F, U4 TL431DBZ, U5 LM211

Commit message: my new version is coming
Parts:
- removed C7: 100nF, Capacitor_SMD:C_1206_3216Metric, symbol Device:C
- removed D1, D2, D3, D4: LED, LED_SMD:LED_1206_3216Metric, symbol Device:LED
- removed J1: Conn_01x03, Connector_PinHeader_2.54mm:PinHeader_1x06_P2.54mm_Vertical, symbol Connector_Generic:Conn_01x06
- removed J3: Conn_01x02_Female, esp-light-box:WG235-2P, symbol Connector:Conn_01x02_Female
- removed Q10, Q13, Q5, Q6, Q9: Q_PMOS_DGS, symbol Device:Q_PMOS_DGS
- removed Q12, Q7: Q_NMOS_DGS, symbol Device:Q_NMOS_DGS
- removed Q15: S8050, Package_TO_SOT_THT:TO-92_Inline, symbol Transistor_BJT:S8050
- removed Q4: Q_P, symbol Device:Q_DUAL_PMOS_G1S2G2D2S1D1
- removed R11, R13, R17, R18, R20, R21, R9: 10K, Resistor_SMD:R_1206_3216Metric, symbol Device:R
- removed R19: 10k, Resistor_SMD:R_1206_3216Metric, symbol Device:R
- removed U4: TL431DBZ, Package_TO_SOT_SMD:SOT-23, symbol Reference_Voltage:TL431DBZ
- added C12, C4: 100nF, Capacitor_SMD:C_0402_1005Metric, symbol Device:C
- added D1: 2.4V, Diode_SMD:D_SOD-323, symbol Device:D_Zener
- added J1: Conn_01x04, Connector_PinHeader_2.54mm:PinHeader_1x04_P2.54mm_Vertical, symbol Connector_Generic:Conn_01x04
- added J3: Conn_01x03_Female, esp-light-box:SolderWire_1x03_2.5x6, symbol Connector:Conn_01x03_Female
- added J5: Conn_01x02, Connector_PinHeader_2.54mm:PinHeader_1x02_P2.54mm_Vertical, symbol Connector_Generic:Conn_01x02
- added Q2, Q6: Q_PMOS_DGS, Package_TO_SOT_SMD:SOT-23-6, symbol Device:Q_DUAL_PMOS_G1S2G2D2S1D1
- added Q5: S8050, Package_TO_SOT_SMD:SOT-23, symbol Transistor_BJT:S8050
- added Q9: Q_NMOS, Package_TO_SOT_SMD:SOT-23, symbol Transistor_FET:2N7002
- added R15: 20K, Resistor_SMD:R_0402_1005Metric, symbol Device:R
- added R3: 10K, Resistor_SMD:R_0402_1005Metric, symbol Device:R
- added R5, R7: 20K, Resistor_SMD:R_0603_1608Metric, symbol Device:R
- added R6: 300, Resistor_SMD:R_0805_2012Metric, symbol Device:R
- C1: footprint (none) -> Capacitor_SMD:C_1206_3216Metric; LCSC (none) -> C12891
- C10: footprint (none) -> Capacitor_SMD:C_0402_1005Metric
- C11: renamed from C9; value 1m -> 220u; footprint (none) -> Capacitor_SMD:CP_Elec_6.3x7.7; LCSC (none) -> C127327
- C2: renamed from C4; footprint Capacitor_SMD:C_1210_3225Metric -> Capacitor_Tantalum_SMD:CP_EIA-3216-18_Kemet-A; symbol Device:C -> Device:CP; LCSC (none) -> C177743
- C3: renamed from C2; value 0.1uF -> 100nF; footprint Capacitor_SMD:C_1206_3216Metric -> Capacitor_SMD:C_0402_1005Metric; LCSC (none) -> C307331
- C5: renamed from C3; footprint Capacitor_SMD:C_1206_3216Metric -> Capacitor_SMD:C_0402_1005Metric; LCSC (none) -> C18047
- C6: renamed from C5; footprint Capacitor_SMD:C_1206_3216Metric -> Capacitor_SMD:C_0402_1005Metric; LCSC (none) -> C15195
- C7: renamed from C6; value 22uF/6.3V -> 47uF/6.3V; footprint Capacitor_SMD:C_1210_3225Metric -> Capacitor_SMD:C_1206_3216Metric; LCSC (none) -> C96123
- C8: footprint Capacitor_SMD:C_1210_3225Metric -> Capacitor_Tantalum_SMD:CP_EIA-3216-18_Kemet-A; symbol Device:C -> Device:CP; LCSC (none) -> C7185
- C9: renamed from C11; value 1u -> 10u; footprint (none) -> Capacitor_SMD:C_0603_1608Metric; LCSC (none) -> C19702
- IC1: footprint QFN50P400X400X80-25N-D -> CP2105-F01-GMR:QFN50P400X400X80-25N-D; LCSC (none) -> C109102
- J4: renamed from J2; footprint Connector_PinHeader_2.54mm:PinHeader_1x03_P2.54mm_Vertical -> esp-light-box:SolderWire_1x03_2.5x6
- L1: footprint Inductor_SMD:L_Abracon_ASPI-0630LR -> Inductor_SMD:L_Sunlord_MWSA0518_5.4x5.2mm; LCSC (none) -> C181721
- Q1: renamed from Q2; footprint (none) -> Package_TO_SOT_SMD:SOT-23; symbol Device:Q_DUAL_NMOS_S1G1D2S2G2D1 -> Transistor_FET:2N7002; LCSC (none) -> C8545
- Q3: value Q_DUAL_PMOS_G1S2G2D2S1D1 -> Q_PMOS_DGS; footprint (none) -> Package_TO_SOT_SMD:SOT-23-6; LCSC (none) -> C148368
- Q3: renamed from Q8; footprint (none) -> Package_TO_SOT_SMD:SOT-23-6; symbol Device:Q_PMOS_DGS -> Device:Q_DUAL_PMOS_G1S2G2D2S1D1; LCSC (none) -> C148368
- Q4: renamed from Q14; footprint Package_TO_SOT_THT:TO-92_Inline -> Package_TO_SOT_SMD:SOT-23; LCSC (none) -> C2146
- Q7: renamed from Q1; LCSC (none) -> C52895
- Q8: renamed from Q11; footprint (none) -> Package_TO_SOT_SMD:TO-252-2; symbol Device:Q_PMOS_DGS -> Transistor_FET:SUD50P04-08; LCSC (none) -> C67281
- R1, R2: value 120 -> 1M; footprint Resistor_SMD:R_1206_3216Metric -> Resistor_SMD:R_0402_1005Metric; LCSC (none) -> C26083
- R10: footprint Resistor_SMD:R_1206_3216Metric -> Resistor_SMD:R_0402_1005Metric; LCSC (none) -> C25895
- R11: renamed from R3; value 1k -> 360; footprint Resistor_SMD:R_1206_3216Metric -> Resistor_SMD:R_1210_3225Metric; LCSC (none) -> C25426
- R12: footprint Resistor_SMD:R_1206_3216Metric -> Resistor_SMD:R_0402_1005Metric; LCSC (none) -> C25744
- R13: renamed from R5; footprint Resistor_SMD:R_1206_3216Metric -> Resistor_SMD:R_0603_1608Metric; LCSC (none) -> C23352
- R14: renamed from R8; footprint Resistor_SMD:R_1206_3216Metric -> Resistor_SMD:R_0603_1608Metric; LCSC (none) -> C25804
- R16: value 10k -> 20K; footprint Resistor_SMD:R_1206_3216Metric -> Resistor_SMD:R_0402_1005Metric; LCSC (none) -> C25765
- R17: renamed from R25; footprint (none) -> Resistor_SMD:R_0402_1005Metric; LCSC (none) -> C25752
- R18: renamed from R26; footprint (none) -> Resistor_SMD:R_0402_1005Metric; LCSC (none) -> C25752
- R21: renamed from R22; footprint (none) -> Resistor_SMD:R_0402_1005Metric
- R22: renamed from R23; footprint (none) -> Resistor_SMD:R_0402_1005Metric; LCSC (none) -> C25774
- R23: renamed from R24; footprint (none) -> Resistor_SMD:R_0402_1005Metric; LCSC (none) -> C25774
- R24: renamed from R14; footprint Resistor_SMD:R_1206_3216Metric -> Resistor_SMD:R_0402_1005Metric; LCSC (none) -> C25744
- R25: renamed from R15; footprint Resistor_SMD:R_1206_3216Metric -> Resistor_SMD:R_0402_1005Metric; LCSC (none) -> C25744
- R4: footprint Resistor_SMD:R_1206_3216Metric -> Resistor_SMD:R_0402_1005Metric; LCSC (none) -> C25741
- R8: renamed from R6; footprint Resistor_SMD:R_1206_3216Metric -> Resistor_SMD:R_0402_1005Metric; LCSC (none) -> C25917
- R9: renamed from R7; footprint Resistor_SMD:R_1206_3216Metric -> Resistor_SMD:R_0402_1005Metric; LCSC (none) -> C25744
- U1: LCSC (none) -> C18921
- U2: renamed from U3; footprint ESP8266:ESP-12E -> RF_Module:ESP-12E; symbol esp-led-box-rescue:ESP-12F-ESP8266 -> RF_Module:ESP-12F
- U3: renamed from U5; footprint (none) -> Package_SO:SOIC-8-1EP_3.9x4.9mm_P1.27mm_EP2.29x3mm; LCSC (none) -> C99580
- U4: renamed from U2; LCSC (none) -> C140319
- renumbered J4 to J2
Connections:
- net LED_PWR is gone; now on net VDD: F1.2
- net +12V: now also Q2.4 (D)
- net +3V3: now also C4.1, J5.1 (Pin_1), R3.1; no longer C10.1, IC1.5 (VIO), IC1.6 (VDD), IC1.7 (REGIN), R21.1
- net +5V: now also Q3.2 (S), Q3.5 (S); no longer Q3.3 (S)
- net BUCK_5V: now also Q3.6 (D)
- net DC_5V: now also Q3.4 (D), Q2.6 (D); no longer Q3.6 (D)
- net DTR: now also Q5.1 (E)
- net GND: now also Q1.2 (S), R1.2, R12.2, R2.2, U2.15 (GND), C12.1, C4.2, D1.2 (A), J3.3 (Pin_3), J5.2 (Pin_2), Q9.2 (S); no longer J2.6 (Shield), Q1.1 (S), Q3.2 (G), Q8.2 (G), R12.1, U2.9 (GND)
- net GPIO0: now also U2.18 (GPIO0), J1.1 (Pin_1); no longer U2.12 (GPIO0)
- net RESET: now also J1.4 (Pin_4), Q5.3 (C)
- net TXD: now also U2.22 (GPIO1/TXD), J1.2 (Pin_2); no longer U2.16 (TXD)
- net VBUS: now also C10.1, IC1.7 (REGIN), R1.1, Q6.5 (S), R5.1; no longer Q3.1 (D)
- net VDC: now also Q8.2 (D), R2.1, J3.1 (Pin_1), J3.2 (Pin_2), R6.1, R7.1; no longer C11.1, Q8.1 (D), R16.1
- net VDD: now also C11.1, J4.3 (Pin_3), R16.1, Q2.2 (S), Q2.5 (S), R15.1; no longer Q3.5 (S)
- net at U2.10 (MISO): no longer R12.2
- net LED_CTRL: now reaches U2.17 (GPIO2)
- net LED_CTRL: now also Q7.2 (S), R24.1
- net RXD: now reaches U2.21 (GPIO3/RXD)
- net RXD: now also R22.2, J1.3 (Pin_3)
- net at U2.3 (EN): now also R3.2
- net DC_VDD: now reaches F1.1
- net DC_VDD: now also Q8.3 (S), Q6.2 (S); no longer J4.3 (Pin_3)
- net ~12V_SEL: now reaches U3.7
- net ~12V_SEL: now also Q1.1 (G), Q3.1 (G), Q2.3 (G), R15.2; no longer Q1.2 (G)
- net at R18.2: now also Q5.2 (B)
- net ~5V_SEL: now reaches R16.2
- net ~5V_SEL: now also Q1.3 (D), Q3.3 (G), Q2.1 (G)
- net at R11.1, U3.3 (-): now also D1.1 (K)
- net GRN_LED: no longer names the net of U2.4 (GPIO16)
- net GRN_LED: no longer R1.1
- net RED_LED: no longer names the net of U2.5 (GPIO14)
- net RED_LED: no longer R2.1
- removed net RXD|CONTROL: Q7.2 (S), R22.2, R24.1, U2.15 (RXD)
- new net: R12.1, U2.16 (GPIO15)
- new net: Q6.4 (D), Q6.6 (D)
- new net: Q9.1 (G), R7.2
- new net VDC_ON: Q6.1 (G), Q6.3 (G), R6.2
- new net V_IO: C12.2, IC1.5 (VIO), IC1.6 (VDD), R21.1
- new net ~VDC_SEL: Q8.1 (G), Q9.3 (D), R5.2
- no-connect marks 26 -> 15
Other:
- moved on the sheet: C1, C10, C11, C3, C5, C6, C7, C9, F1, IC1, J2, J4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

Commit message: kek forgot it
Parts:
- R21: LCSC (none) -> C25900
Changed lines of the file:
@@
 F 2 "Resistor_SMD:R_0402_1005Metric" V 13230 8650 50  0001 C CNN
 F 3 "~" H 13300 8650 50  0001 C CNN
+F 4 "C25900" H 13300 8650 50  0001 C CNN "LCSC"
 	1    13300 8650
 	-1   0    0    1

Commit message: another kek
Connections:
- net +3V3: now also J5.2 (Pin_2); no longer J5.1 (Pin_1)
- net GND: now also J5.1 (Pin_1); no longer J5.2 (Pin_2)
- net RESET: now also J1.2 (Pin_2); no longer J1.4 (Pin_4)
- net TXD: now also J1.4 (Pin_4); no longer J1.2 (Pin_2)
Changed lines of the file:
@@
 	1    0    0    1
 $EndComp
+Text Label 9850 8700 2    50   ~ 0
+GPIO0
+Text Label 9850 8600 2    50   ~ 0
+RESET
 Text Label 9850 8400 2    50   ~ 0
-GPIO0
-Text Label 9850 8700 2    50   ~ 0
-RESET
+TXD
 Text Label 9850 8500 2    50   ~ 0
-TXD
-Text Label 9850 8600 2    50   ~ 0
 RXD
 $Comp
@@
 L Connector_Generic:Conn_01x02 J5
 U 1 1 624C44C8
-P 10050 9050
-F 0 "J5" H 10130 9042 50  0000 L CNN
-F 1 "Conn_01x02" H 10130 8951 50  0000 L CNN
-F 2 "Connector_PinHeader_2.54mm:PinHeader_1x02_P2.54mm_Vertical" H 10050 9050 50  0001 C CNN
-F 3 "~" H 10050 9050 50  0001 C CNN
-	1    10050 9050
-	1    0    0    -1
+P 10050 9150
+F 0 "J5" H 10130 9142 50  0000 L CNN
+F 1 "Conn_01x02" H 10130 9051 50  0000 L CNN
+F 2 "Connector_PinHeader_2.54mm:PinHeader_1x02_P2.54mm_Vertical" H 10050 9150 50  0001 C CNN
+F 3 "~" H 10050 9150 50  0001 C CNN
+	1    10050 9150
+	1    0    0    1
 $EndComp
 $Comp
 L Connector_Generic:Conn_01x04 J1
 U 1 1 624C9F56
-P 10050 8500
-F 0 "J1" H 10130 8492 50  0000 L CNN
-F 1 "Conn_01x04" H 10130 8401 50  0000 L CNN
-F 2 "Connector_PinHeader_2.54mm:PinHeader_1x04_P2.54mm_Vertical" H 10050 8500 50  0001 C CNN
-F 3 "~" H 10050 8500 50  0001 C CNN
-	1    10050 8500
-	1    0    0    -1
+P 10050 8600
+F 0 "J1" H 10130 8592 50  0000 L CNN
+F 1 "Conn_01x04" H 10130 8501 50  0000 L CNN
+F 2 "Connector_PinHeader_2.54mm:PinHeader_1x04_P2.54mm_Vertical" H 10050 8600 50  0001 C CNN
+F 3 "~" H 10050 8600 50  0001 C CNN
+	1    10050 8600
+	1    0    0    1
 $EndComp
 $EndSCHEMATC
