File: esp-led-box.sch (KiCad schematic (older format))
At the start: 57 parts, among them IC1 CP2105-F01-GMR, J1 Conn_01x04, J2 USB_B_Micro, J3 Conn_01x03_Female, J4 Conn_01x03_Female, J5 Conn_01x02, Q1 Q_NMOS, Q2 Q_PMOS_DGS, Q3 Q_PMOS_DGS, Q4 S8050, Q5 S8050, Q6 Q_PMOS_DGS, Q7 BSS138, Q8 Q_PMOS_DGS, Q9 Q_NMOS, U1 MP2307, U2 ESP-12F, U3 LM211, U4 LM3940

Commit message: will I ever stop?
Parts:
- removed C2: 10uF, Capacitor_Tantalum_SMD:CP_EIA-3216-18_Kemet-A, symbol Device:CP
- removed R14: 10K, Resistor_SMD:R_0603_1608Metric, symbol Device:R
- added C?: 22uF 6.3V, Capacitor_SMD:C_0603_1608Metric, symbol Device:C
- added R13: 10K, Resistor_SMD:R_0402_1005Metric, symbol Device:R
- C1: value 10u/25V -> 22u/25V; footprint Capacitor_SMD:C_1206_3216Metric -> Capacitor_SMD:C_0805_2012Metric; LCSC C12891 -> C45783
- C7: value 47uF/6.3V -> 22uF 6.3V; footprint Capacitor_SMD:C_1206_3216Metric -> Capacitor_SMD:C_0603_1608Metric; LCSC C96123 -> C59461
- C8: value 33uF -> 100uF; footprint Capacitor_Tantalum_SMD:CP_EIA-3216-18_Kemet-A -> Capacitor_Tantalum_SMD:CP_EIA-3528-21_Kemet-B; LCSC C7185 -> C16133
- D1: value 2.4V -> 5.6V; footprint Diode_SMD:D_SOD-323 -> Diode_SMD:D_MiniMELF; LCSC C17285 -> C8062
- Q1, Q9: value Q_NMOS -> 2N7002
- Q7: value BSS138 -> 2N7002; LCSC C52895 -> C8545
- R11: value 360 -> 1K; footprint Resistor_SMD:R_1210_3225Metric -> Resistor_SMD:R_0603_1608Metric; LCSC C25426 -> C21190
- R14: renamed from R13; value 24K -> 22K; footprint Resistor_SMD:R_0603_1608Metric -> Resistor_SMD:R_0402_1005Metric; LCSC C23352 -> C25768
Connections:
- net BUCK_5V: now also C?.1
- net GND: now also R14.2, C?.2
- net VDD: now also R13.1; no longer R14.1
- net at U3.2 (+): now also R14.1, R13.2; no longer R14.2
Other:
- moved on the sheet: C4, R12, R14, R3, U2, U4

Commit message: finally we are done
Parts:
- gave numbers to parts that had none: 1
- renumbered C12 to C10, C10 to C11, C11 to C12, C3 to C2, C5 to C3, C8 to C4, C6 to C5, C4 to C6, J5 to J2, J2 to J3, J3 to J4, J4 to J5, Q9 to Q1, Q1 to Q2, Q2 to Q3, Q3 to Q4, Q4 to Q5, Q5 to Q6, Q6 to Q7, Q7 to Q8, Q8 to Q9, R3 to R10, R13 to R12, R14 to R13, R15 to R14, R12 to R15, R21 to R19, R22 to R20, R23 to R21, R24 to R22, R25 to R23, R4 to R3, R5 to R4, R6 to R5, R7 to R6, R8 to R7, R9 to R8, R10 to R9, U4 to U1, U1 to U2, U2 to U3, U3 to U4
